Commit message: Add SAKE mounts and configurations for single, double, and triple grippers

File: ezgripper_description/urdf/materials.urdf.xacro (robot description, xacro)
@@ -1,4 +1,4 @@
 <?xml version="1.0"?>
-<robot name="ezgripper_single_mount" xmlns:xacro="http://ros.org/wiki/xacro">
+<robot xmlns:xacro="http://ros.org/wiki/xacro">
   <material name="black">
     <color rgba="0.0 0.0 0.0 1.0"/>
@@ -10,3 +10,6 @@
     <color rgba="0.5 0.5 0.5 1"/>
   </material>
+  <material name="white">
+    <color rgba="1.0 1.0 1.0 1.0"/> <!-- RGBA: Red, Green, Blue, Alpha (transparency) -->
+  </material>
 </robot>
