Commit message: Improve triple gripper integration with proper material definitions and joint state publishing
- Added robot_components.yaml for joint configuration
- Added gripper_joint_publisher and gripper_static_tf_publisher
- Fixed material definitions in SAKE_triple_mount.urdf.xacro
- Added integration launch files for combining with other robot components
- Updated URDF files for better compatibility
- Added materials.xacro for standardized material definitions

File: ezgripper_description/urdf/SAKE_single_mount.urdf.xacro (robot description, xacro)
@@ -1,4 +1,6 @@
 <?xml version="1.0" encoding="UTF-8"?>
 <robot name="SAKE_single_mount" xmlns:xacro="http://ros.org/wiki/xacro">
+    <!-- Include centralized material definitions (properties only) -->
+    <xacro:include filename="$(find ezgripper_description)/urdf/materials.xacro" />
 	<xacro:macro name="SAKE_single_mount" params="prefix parent_link *origin">
 		<!-- links -->
@@ -16,5 +18,5 @@
 					<mesh filename="file://$(find ezgripper_description)/meshes/visual/SAKE_Single_Mount.stl"/>
 				</geometry>
-				<material name="blue"/>
+				<material name="ezgripper_blue"/>
 			</visual>
 			<collision>

File: ezgripper_description/urdf/SAKE_triple_mount.urdf.xacro (robot description, xacro)
@@ -14,12 +14,12 @@
 				<origin rpy="0 0 0" xyz="0.0 0.0 0.0"/>
 				<geometry>
-					<mesh filename="file://$(find ezgripper_description)/meshes/visual/SAKE_Triple_Mount.stl"/>
+					<mesh filename="package://ezgripper_description/meshes/visual/SAKE_Triple_Mount.stl"/>
 				</geometry>
-				<material name="blue"/>
+				<material name="ezgripper_blue"/>
 			</visual>
 			<collision>
 				<origin rpy="0 0 0" xyz="0.0 0.0 0.0"/>
 				<geometry>
-					<mesh filename="file://$(find ezgripper_description)/meshes/collision/SAKE_Triple_Mount.stl"/>
+					<box size="0.05 0.05 0.15"/>
 				</geometry>
 			</collision>
@@ -29,5 +29,5 @@
 			</inertial>
 		</link>
-		<gazebo reference="${prefix}_ezgripper_mount">
+		<gazebo reference="${prefix}_ezgripper_to_mount">
 			<material>Gazebo/Blue</material>
 		</gazebo>

File: ezgripper_description/urdf/ezgripper_single.urdf.xacro (robot description, xacro)
@@ -1,4 +1,6 @@
 <?xml version="1.0" encoding="UTF-8"?>
 <robot name="ezgripper_single" xmlns:xacro="http://ros.org/wiki/xacro">
+    <!-- Include centralized material definitions (properties only) -->
+    <xacro:include filename="$(find ezgripper_description)/urdf/materials.xacro" />
 	<xacro:macro name="ezgripper_single" params="prefix parent_link *origin">
 		<!-- links -->
@@ -19,12 +21,12 @@
 				<origin xyz="0.0 0 0" rpy="0 0 0"/>
 				<geometry>
-					<mesh filename="file://$(find ezgripper_description)/meshes/visual/SAKE_Palm_IM.stl"/>
-				</geometry>
-				<material name="blue"/>
+					<mesh filename="package://ezgripper_description/meshes/visual/SAKE_Palm_IM.stl"/>
+				</geometry>
+				<material name="ezgripper_blue"/>
 			</visual>
 			<collision>
 				<origin xyz="0.0 0 0" rpy="0 0 0"/>
 				<geometry>
-					<mesh filename="file://$(find ezgripper_description)/meshes/collision/SAKE_Palm_IM.stl"/>
+					<box size="0.04 0.04 0.04"/>
 				</geometry>
 			</collision>
@@ -59,12 +61,12 @@
 				<origin xyz="0 0 0" rpy="0 0 0"/>
 				<geometry>
-					<mesh filename="file://$(find ezgripper_description)/meshes/visual/SAKE_Finger_L1_IM.stl"/>
-				</geometry>
-				<material name="grey"/>
-			</visual>
-			<collision>
-				<origin xyz="0 0 0" rpy="0 0 0"/>
-				<geometry>
-					<mesh filename="file://$(find ezgripper_description)/meshes/collision/SAKE_Finger_L1_IM.stl"/>
+					<mesh filename="package://ezgripper_description/meshes/visual/SAKE_Finger_L1_IM.stl"/>
+				</geometry>
+				<material name="ezgripper_grey"/>
+			</visual>
+			<collision>
+				<origin xyz="0 0 0" rpy="0 0 0"/>
+				<geometry>
+					<box size="0.03 0.01 0.03"/>
 				</geometry>
 			</collision>
@@ -83,12 +85,12 @@
 				<origin xyz="0 0 0" rpy="0 0 0"/>
 				<geometry>
-					<mesh filename="file://$(find ezgripper_description)/meshes/visual/SAKE_Finger_L2_IM.stl"/>
-				</geometry>
-				<material name="grey"/>
-			</visual>
-			<collision>
-				<origin xyz="0 0 0" rpy="0 0 0"/>
-				<geometry>
-					<mesh filename="file://$(find ezgripper_description)/meshes/collision/SAKE_Finger_L2_IM.stl"/>
+					<mesh filename="package://ezgripper_description/meshes/visual/SAKE_Finger_L2_IM.stl"/>
+				</geometry>
+				<material name="ezgripper_grey"/>
+			</visual>
+			<collision>
+				<origin xyz="0 0 0" rpy="0 0 0"/>
+				<geometry>
+					<box size="0.03 0.01 0.03"/>
 				</geometry>
 			</collision>
@@ -107,12 +109,12 @@
 				<origin xyz="0 0 0" rpy="0 0 0"/>
 				<geometry>
-					<mesh filename="file://$(find ezgripper_description)/meshes/visual/SAKE_Finger_Pad_IM.stl"/>
-				</geometry>
-				<material name="grey"/>
-			</visual>
-			<collision>
-				<origin xyz="0 0 0" rpy="0 0 0"/>
-				<geometry>
-					<mesh filename="file://$(find ezgripper_description)/meshes/collision/SAKE_Finger_Pad_IM.stl"/>
+					<mesh filename="package://ezgripper_description/meshes/visual/SAKE_Finger_Pad_IM.stl"/>
+				</geometry>
+				<material name="ezgripper_grey"/>
+			</visual>
+			<collision>
+				<origin xyz="0 0 0" rpy="0 0 0"/>
+				<geometry>
+					<box size="0.02 0.01 0.02"/>
 				</geometry>
 			</collision>

File: ezgripper_description/urdf/ezgripper_single_with_mount.urdf.xacro (robot description, xacro)
@@ -1,4 +1,6 @@
 <?xml version="1.0" encoding="UTF-8"?>
 <robot name="ezgripper_single_with_mount" xmlns:xacro="http://ros.org/wiki/xacro">
+    <!-- Include centralized material definitions (properties only) -->
+    <xacro:include filename="$(find ezgripper_description)/urdf/materials.xacro" />
     <xacro:macro name="ezgripper_single_with_mount" params="prefix parent_link *origin">
 	<!-- Include the gripper and mount files -->

File: ezgripper_description/urdf/ezgripper_single_with_mount_standalone.urdf.xacro (robot description, xacro)
@@ -1,8 +1,11 @@
 <?xml version="1.0" encoding="UTF-8"?>
 <robot name="ezgripper_single_mount_instantiation" xmlns:xacro="http://ros.org/wiki/xacro">
+    <!-- Include centralized material definitions -->
+    <xacro:include filename="$(find ezgripper_description)/urdf/materials.xacro" />
+    <xacro:define_ezgripper_materials />
     <xacro:property name="prefix" value="left" />
     <xacro:property name="ezgripper_offset_x" value="0.00"/>
     <xacro:property name="ezgripper_offset_y" value="0.0"/>
-    <xacro:property name="ezgripper_offset_z" value="0.0"/>
+    <xacro:property name="ezgripper_offset_z" value="0.21"/>
     <xacro:include filename="ezgripper_single_with_mount.urdf.xacro" />
     <!-- Instantiate the gripper and mount assembly with specified parameters -->
@@ -21,5 +24,5 @@
             </geometry>
             <origin rpy="0 0 0" xyz="0 0 0.21"/>
-            <material name="black"/>
+            <material name="ezgripper_black"/>
         </visual>
         <collision>

File: ezgripper_description/urdf/ezgripper_triple_with_mount.urdf.xacro (robot description, xacro)
@@ -2,6 +2,6 @@
 <robot name="ezgripper_triple_with_mount" xmlns:xacro="http://ros.org/wiki/xacro">
   <xacro:macro name="ezgripper_triple_with_mount" params="prefix parent_link *origin">
-    <xacro:property name="gripper_spacing" value="0.068"/>  <!-- Gripper separation in mm -->
-    <xacro:property name="gripper_offset" value="0.01254"/>   <!-- Gripper offset in the positive X direction from the mount in mm single = 16mm, double and triple = 12.54-->
+    <xacro:property name="gripper_spacing" value="0.068"/>  <!-- Gripper separation in m (6.8cm) -->
+    <xacro:property name="gripper_offset" value="0.01254"/>   <!-- Gripper offset in the positive X direction from the mount in m (1.254cm) -->
     <!-- Include the gripper and mount files -->
     <xacro:include filename="$(find ezgripper_description)/urdf/SAKE_triple_mount.urdf.xacro" />

File: ezgripper_description/urdf/ezgripper_triple_with_mount_standalone.urdf.xacro (robot description, xacro)
@@ -1,13 +1,16 @@
 <?xml version="1.0" encoding="UTF-8"?>
 <robot name="ezgripper_triple_mount_instantiation" xmlns:xacro="http://ros.org/wiki/xacro">
+    <!-- Include centralized material definitions -->
+    <xacro:include filename="$(find ezgripper_description)/urdf/materials.xacro" />
+    <xacro:define_ezgripper_materials />
     <xacro:property name="prefix" value="left" />
     <xacro:property name="ezgripper_offset_x" value="0.00"/>
     <xacro:property name="ezgripper_offset_y" value="0.0"/>
-    <xacro:property name="ezgripper_offset_z" value="0.0"/>
+    <xacro:property name="ezgripper_offset_z" value="0.21"/>
     <xacro:include filename="ezgripper_triple_with_mount.urdf.xacro" />
     <!-- Instantiate the gripper and mount assembly with specified parameters -->
-	<xacro:ezgripper_triple_with_mount prefix="${prefix}" parent_link="base_link">
-		<origin xyz="${ezgripper_offset_x} ${ezgripper_offset_y} ${ezgripper_offset_z}" rpy="0 0 0"/>
-	</xacro:ezgripper_triple_with_mount>
+    <xacro:ezgripper_triple_with_mount prefix="${prefix}" parent_link="base_link">
+        <origin xyz="${ezgripper_offset_x} ${ezgripper_offset_y} ${ezgripper_offset_z}" rpy="0 0 0"/>
+    </xacro:ezgripper_triple_with_mount>
     <link name="world"/>
     <joint name="fixed" type="fixed">
@@ -21,5 +24,5 @@
             </geometry>
             <origin rpy="0 0 0" xyz="0 0 0.21"/>
-            <material name="black"/>
+            <material name="ezgripper_black"/>
         </visual>
         <collision>
